File: doc/schematic/C64UsbKeyboard/C64UsbKeyboard.kicad_sch (KiCad schematic)
At the start: 9 parts, among them J1 USB_Plug, J3 Debug, J5 C64Keyboard, U2 YAAJ_BluePill_Part_Like

Commit message: First working version.
Parts:
- added D10, D11, D2, D4, D5, D6, D7, D8, D9: 1N4148, Diode_THT:D_DO-35_SOD27_P7.62mm_Horizontal, symbol Diode:1N4148
- added J2: Add_Keys, symbol Connector_Generic:Conn_01x04
Connections:
- net GND: no longer J5.1 (Pin_1)
- net Row_0: now also D11.1 (K), J2.1 (Pin_1); no longer J5.12 (Pin_12)
- net Row_1: now also D10.1 (K), J2.4 (Pin_4); no longer J5.11 (Pin_11)
- net Row_2: now also D9.1 (K); no longer J5.10 (Pin_10)
- net Row_3: now also D8.1 (K); no longer J5.9 (Pin_9)
- net Row_4: now also D7.1 (K); no longer J5.8 (Pin_8)
- net Row_5: now also D6.1 (K); no longer J5.7 (Pin_7)
- net Row_6: now also D5.1 (K); no longer J5.6 (Pin_6)
- net Row_7: now also D4.1 (K); no longer J5.5 (Pin_5)
- net Col_I: now reaches U2.2 (PB13)
- net Col_I: now also J5.1 (Pin_1)
- net Row_8: now reaches U2.3 (PB14)
- net Row_8: now also D2.1 (K)
- net Restore_0: no longer names the net of U2.33 (PB0)
- net Restore_0: no longer J5.3 (Pin_3)
- new net: D10.2 (A), J5.11 (Pin_11)
- new net: D2.2 (A), J5.3 (Pin_3)
- new net: D8.2 (A), J5.9 (Pin_9)
- new net: D9.2 (A), J5.10 (Pin_10)
- new net: D11.2 (A), J5.12 (Pin_12)
- new net: D4.2 (A), J5.5 (Pin_5)
- new net: D5.2 (A), J5.6 (Pin_6)
- new net: D6.2 (A), J5.7 (Pin_7)
- new net: D7.2 (A), J5.8 (Pin_8)
- new net Restore_A: J2.2 (Pin_2), J2.3 (Pin_3)
Other:
- note added: "Additional Keys Row0 / ColI = F12 (Menu) Row1 / ColI = PAGE_UP (Tape Play)"
- note added: "To I2C of Companion Board Not used at the moment."
- note added: "USB Cable Not necessary, if Bluepill plug is used."
- note removed: "To I2C of Companion Board"
- note removed: "USB Cable"
- moved on the sheet: J1, J5
